Commit message: initial configuration files and top_platform and one top_ball shows up

File: urdf/stewart_platform.urdf (robot description, URDF)
Before this commit: robot stewart, 7 links, 6 joints
Links:
- removed link bottom_ball1_link
- removed link piston1_cylinder_link
- removed link piston1_shaft_link
- removed link top_ball1_link_vert
- removed link world
- link platform_link: mass 1.0 -> None; geometry visual cylinder length=0.1 radius=1.0
- link top_ball1_link_hor: mass 0.1 -> None; geometry visual sphere radius=0.05
Joints:
- removed joint initial
- removed joint piston1_bottom_pitch_joint
- removed joint piston1_prismatic_joint
- removed joint piston1_top_pitch_joint
- removed joint top_ball1_joint_vert
- joint top_ball1_joint_hor: axis 1 0 0 -> 0 0 1

Commit message: swapped origin order of link and joint for ball joints -- now working, supposedly

File: urdf/stewart_platform.urdf (robot description, URDF)
Before this commit: robot stewart, 2 links, 1 joints
Joints:
- joint top_ball1_joint_hor: origin xyz=0 0 0 rpy=0 0 0 -> xyz=-0.6423496169447003 0.4872237367072718 2.075 rpy=0 0 2.0945

Commit message: black shaft is rotated wrong?

File: urdf/stewart_platform.urdf (robot description, URDF)
Before this commit: robot stewart, 2 links, 1 joints
Links:
- added link piston1_shaft_link; visual cylinder length=1.9291197998702527 radius=0.05
- added link top_ball1_link_vert; visual sphere radius=0.05
Joints:
- added joint piston1_top_pitch_joint: type revolute, parent top_ball1_link_vert, child piston1_shaft_link, origin xyz=0 0 -0.9645598999351264 rpy=0 0 0, axis 1 0 0, limit lower=-0.786 upper=0.786 effort=-1.0 velocity=-1.0
- added joint top_ball1_joint_vert: type revolute, parent top_ball1_link_hor, child top_ball1_link_vert, origin xyz=0 0 0 rpy=0 0 0, axis 0 1 0, limit lower=-0.786 upper=0.786 effort=-1.0 velocity=0.1

Commit message: Issue: Prismatic is not 'parent' to any other joints -> how to make it move the other stuff

File: urdf/stewart_platform.urdf (robot description, URDF)
Before this commit: robot stewart, 4 links, 3 joints
Links:
- added link piston1_cylinder_link, mass 0.1; visual cylinder length=1.9291197998702527 radius=0.1
Joints:
- added joint piston1_prismatic_joint: type prismatic, parent piston1_shaft_link, child piston1_cylinder_link, origin xyz=0 0 0 rpy= 0 0 0, axis 0 0 -1, limit lower=0 upper=1.9291197998702527 effort=-1.0 velocity=1.0
